File: template/eaglecad/mezza.brd (EAGLE design)
At the start: 85 x 54 mm, 3 parts, among them J1 55510-140LF, J2 61083-063402LF

Commit message: v1 board
Parts:
- added ANT1, ANT2: (no value), BeagleBone_Black_Wireless:GHI-CONNECTORS_U.FL-R-SMT-1
- added C1, C10, C11, C14, C15, C2, C3, C6, C7, C8, C9: 0.1uF, SparkFun-Capacitors:0603
- added C12, C13: 0.1uF, resistor:C0603
- added C16, C17, C18: (no value), resistor:C1206
- added C19, C4: 10nF, rcl:C0603
- added C5: 0.1uF, rcl:C0603
- added D1, D2, D3, D4: WHITE, SparkFun-LED:LED-0603
- added D10, D5, D7, D8: RED, SparkFun-LED:LED-0603
- added D6: ASMT-YTD7-0AA02, ASMT-YTD7-0AA02:LED_ASMT-YTD7-0AA02
- added D9: (no value), diode:SMBJ
- added F1: 2920L185DR, 2920L200:SMD050F
- added J3, J4, J6, J7: SM04B-GHS-TB(LF)(SN)-, SM04B-GHS-TB_LF__SN_-:JST_SM04B-GHS-TB(LF)(SN)-
- added J5: 22-05-7028-02, con-molex:7395-02
- added J8: SM06B-GHS-TB(LF)(SN), SM06B-GHS-TB_LF__SN_:JST_SM06B-GHS-TB(LF)(SN)
- added PS1: TSR_2-24120, TSR_2-24120:CONV_TSR_2-24120
- added R1, R13, R14, R2, R5: 10k, rcl:R0603
- added R10, R11, R3, R4, R9: (no value), resistor:R0603
- added R12, R15, R16, R17, R18, R19, R20, R21, R6, R7, R8: 1k, rcl:R0603
- added S1: (no value), SparkFun-Switches:JOYSTICK_MINI
- added S2: MOMENTARY-SWITCH-SPST-SMD-6.2MM-TALL, SparkFun-Switches:TACTILE_SWITCH_SMD_6.2MM_TALL
- added TP1, TP2, TP3, TP4, TP5, TP6, TP7: TEST-POINT3X4, SparkFun-Connectors:PAD.03X.04
- added U$1: SSD1306, ssd1306_oled:128_32_OLED
- added U$2: THN15-2422/3, traco:TRACOTHN
- added U1: BME680, BME680:LGA-8
- added U2, U4: PCA9632DP2,118, PCA9632DP2_118:SOP50P490X110-10N
- added U3, U6, U8: (no value), adafruit:VFSOP-8
- added U5: INA260AIPWR, INA260AIPWR:SOP65P640X120-16N
- added U7: TPS73633DBVTG4, TPS73633:SOT23-5
- added U9: TXB0104, SparkFun-IC-Comms:TSSOP14
- added X1: WIFI_1, adafruit:SMA_EDGELAUNCH
- added X2: WIFI_2, adafruit:SMA_EDGELAUNCH
Connections:
- new net +12V: PS1.3, R7.2, TP3.P$1, U$2.3, U5.1, U5.12, U5.2, U5.3
- new net +3V3: C1.1, C11.1, C14.1, C15.1, C2.1, C4.1, C7.1, C9.1, R12.2, R13.2, R14.2, TP4.P$1, U$1.3V3, U1.2, U1.6, U1.8, U2.10, U2.5, U2.7, U3.P$7, U4.10, U6.P$7, U7.5, U8.P$7
- new net CS: J8.3, U9.12
- new net EXT_VIN: D9.C, F1.2, J5.1
- new net MISO: J8.4, U9.11
- new net MOSI: J8.5, U9.10
- new net N$1: D7.C, R5.1, U5.7
- new net N$10: ANT2.SIG, X2.P
- new net N$11: D6.4, R21.1
- new net N$12: ANT2.GND1, ANT2.GND2, X2.GND@1, X2.GND@2, X2.GND@3, X2.GND@4
- new net N$13: D5.A, R7.1
- new net N$14: ANT1.GND1, ANT1.GND2, X1.GND@1, X1.GND@2, X1.GND@3, X1.GND@4
- new net N$15: D8.A, R8.1
- new net N$16: C19.1, U7.4
- new net N$17: D10.A, R12.1
- new net N$2: ANT1.SIG, X1.P
- new net N$21: D1.C, U2.1
- new net N$22: D2.C, U2.2
- new net N$23: J3.2, U3.P$8
- new net N$24: J3.3, U3.P$1
- new net N$25: D4.C, U2.3
- new net N$26: D3.C, U2.4
- new net N$27: F1.1, PS1.1, TP2.P$1, U$2.1, U$2.6
- new net N$28: D6.1, U4.3
- new net N$29: D6.2, U4.2
- new net N$3: D1.A, R15.1
- new net N$30: D6.3, U4.1
- new net N$31: J4.2, U8.P$8
- new net N$34: J4.3, U8.P$1
- new net N$4: D2.A, R16.1
- new net N$5: D4.A, R17.1
- new net N$6: D3.A, R18.1
- new net N$7: D7.A, R6.2
- new net N$8: D6.6, R19.1
- new net N$9: D6.5, R20.1
- new net SCLK: J8.2, U9.13
- new net SCL_3V3: J6.2, J7.2, R13.1, TP7.P$1, U$1.SCL, U1.4, U2.8, U4.8, U5.9, U6.P$1
- new net SDA_3V3: J6.3, J7.3, R14.1, TP6.P$1, U$1.SDA, U1.3, U2.9, U4.9, U5.8, U6.P$8
- net +1V8: now also C10.1, C12.1, C6.1, C8.1, R1.2, R10.2, R11.2, R2.2, R3.2, R4.2, R9.2, TP1.P$1, U3.P$3, U3.P$6, U6.P$3, U6.P$6, U8.P$3, U8.P$6, U9.1, U9.8
- net +5V: now also C13.1, C3.1, C5.1, J3.1, J4.1, J6.1, J7.1, J8.1, R15.2, R16.2, R17.2, R18.2, R19.2, R20.2, R21.2, R5.2, R6.1, TP5.P$1, U5.10, U7.1, U7.3, U9.14
- net GND: now also C1.2, C10.2, C11.2, C12.2, C13.2, C14.2, C15.2, C16.2, C17.2, C18.2, C19.2, C2.2, C3.2, C4.2, C5.2, C6.2, C7.2, C8.2, C9.2, D10.C, D5.C, D8.C, D9.A, J3.4, J3.SH1, J3.SH2, J4.4, J4.SH1, J4.SH2, J5.2, J6.4, J6.SH1, J6.SH2, J7.4, J7.SH1, J7.SH2, J8.6, J8.S1, J8.S2, PS1.2, S1.GND, S2.B2, U$1.GND, U$2.2, U$2.5, U1.1, U1.5, U1.7, U2.6, U4.5, U4.6, U4.7, U5.11, U5.4, U5.5, U5.6, U6.P$2, U7.2, U9.7
- net GPIO-G: now also R10.1, S1.B
- net GPIO-I: now also R9.1, S1.C
- net GPIO-J: now also R4.1, S1.D
- net GPIO-K: now also R3.1, S1.A
- net GPIO-L: now also R11.1, S1.CTR
- net I2C1_SCL: now also R1.1, U6.P$4
- net I2C1_SDA: now also R2.1, U6.P$5
- net RST_BTN_N: now also S2.A2
- net SPI0_CS: now also U9.3
- net SPI0_DIN: now also U9.4
- net SPI0_DOUT: now also U9.2
- net SPI0_SCLK: now also U9.5
- net SYS_DCIN: now also C16.1, C17.1, C18.1, R8.2, U5.14, U5.15, U5.16
- net UART0_RXD: now also U3.P$4
- net UART0_TXD: now also U3.P$5
- net UART1_RXD: now also U8.P$4
- net UART1_TXD: now also U8.P$5
Routing:
- net +5V: track 0.00 -> 196.3 mm, vias 0 -> 10
- net +3V3: track 0.00 -> 158.1 mm, vias 0 -> 7
- net SDA_3V3: track 0.00 -> 151.5 mm, vias 0 -> 10
- net SCL_3V3: track 0.00 -> 145.4 mm, vias 0 -> 10
- net +1V8: track 0.00 -> 110.1 mm, vias 0 -> 11
- net GPIO-J: track 0.00 -> 39.9 mm, vias 0 -> 1
- net GPIO-G: track 0.00 -> 39.0 mm, vias 0 -> 1
- net N$27: track 0.00 -> 34.8 mm
- net GPIO-L: track 0.00 -> 25.1 mm, vias 0 -> 1
- net I2C1_SDA: track 0.00 -> 23.6 mm, vias 0 -> 1
- net N$12: track 0.00 -> 22.9 mm, vias 0 -> 2
- net I2C1_SCL: track 0.00 -> 21.6 mm, vias 0 -> 2
- net GPIO-I: track 0.00 -> 21.6 mm, vias 0 -> 1
- net N$14: track 0.00 -> 19.7 mm, vias 0 -> 2
- net UART1_TXD: track 0.00 -> 19.0 mm, vias 0 -> 1
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- added copper zone on layer 1, net +12V
- added copper zone on layer 1, net GND
- added copper zone on layer 16, net GND
- added copper zone on layer 1, net SYS_DCIN
- added copper zone on layer 16, net SYS_DCIN
Other:
- board text added: "+"
- board text added: "+5V"
- board text added: "-"
- board text added: "12V"
- board text added: "1V8"
- board text added: "1V8 PULLUP"
- board text added: "2020-JVM-R1"
- board text added: "3V3"
- board text added: "3V3 LDO"
- board text added: "3V3 Logic!"
- board text added: "3V3 PULLUP"
- board text added: "5V"
- board text added: "96 Boards Carrier"
- board text added: "CS"
- board text added: "EXT VIN"
- board text added: "GND"
- board text added: "INA260"
- board text added: "Input: +15-33V (4-6S)"
- board text added: "LJMU Astro Eco"
- board text added: "MISO"
- board text added: "MOSI"
- board text added: "PCA9632"
- board text added: "Power Monitor"
- board text added: "RESET"
- board text added: "RGB"
- board text added: "RX0"
- board text added: "RX1"
- board text added: "SCL"
- board text added: "SCLK"
- board text added: "SDA"
- board text added: "SYS DCIN"
- board text added: "TPS73633"
- board text added: "TX0"
- board text added: "TX1"
- board text added: "TXS0102"
- board text added: "UART0"
- board text added: "UART1"
- board text added: "WARN"
- board text removed: "Mezzanine Template"
