File: template/eaglecad/mezza.sch (EAGLE design)
At the start: 3 parts, among them J1 55510-140LF, J2 61083-063402LF

Commit message: v1 board
Parts:
- added ANT1, ANT2: (no value), BeagleBone_Black_Wireless:GHI-CONNECTORS_U.FL-R-SMT-1
- added C1, C10, C11, C14, C15, C2, C3, C6, C7, C8, C9: 0.1uF, SparkFun-Capacitors:0.1UF-0603-25V-(+80/-20%)
- added C12, C13: 0.1uF, resistor:C-EUC0603
- added C16, C17, C18: (no value), resistor:C-EUC1206
- added C19, C4: 10nF, rcl:C-EUC0603
- added C5: 0.1uF, rcl:C-EUC0603
- added D1, D2, D3, D4: WHITE, SparkFun-LED:LED-WHITE0603
- added D10, D5, D7, D8: RED, SparkFun-LED:LED-RED0603
- added D6: ASMT-YTD7-0AA02, ASMT-YTD7-0AA02:ASMT-YTD7-0AA02
- added D9: (no value), diode:SUPPRESSOR-SMBJ
- added F1: 2920L185DR, 2920L200:2920L200
- added J3, J4, J6, J7: SM04B-GHS-TB(LF)(SN)-, SM04B-GHS-TB_LF__SN_-:SM04B-GHS-TB(LF)(SN)-
- added J5: 22-05-7028-02, con-molex:22-05-7028-02
- added J8: SM06B-GHS-TB(LF)(SN), SM06B-GHS-TB_LF__SN_:SM06B-GHS-TB(LF)(SN)
- added PS1: TSR_2-24120, TSR_2-24120:TSR_2-24120
- added R1, R13, R14, R2, R5: 10k, rcl:R-EU_R0603
- added R10, R11, R3, R4, R9: (no value), resistor:R-EU_R0603
- added R12, R15, R16, R17, R18, R19, R20, R21, R6, R7, R8: 1k, rcl:R-EU_R0603
- added S1: (no value), SparkFun-Switches:JOYSTICK_MINI
- added S2: MOMENTARY-SWITCH-SPST-SMD-6.2MM-TALL, SparkFun-Switches:MOMENTARY-SWITCH-SPST-SMD-6.2MM-TALL
- added TP1, TP2, TP3, TP4, TP5, TP6, TP7: TEST-POINT3X4, SparkFun-Connectors:TEST-POINT3X4
- added U$1: SSD1306, ssd1306_oled:SSD1306
- added U$2: THN15-2422/3, traco:THN15-2411
- added U1: BME680, BME680:BME680
- added U2, U4: PCA9632DP2,118, PCA9632DP2_118:PCA9632DP2,118
- added U3, U6, U8: (no value), adafruit:TXS0102
- added U5: INA260AIPWR, INA260AIPWR:INA260AIPWR
- added U7: TPS73633DBVTG4, TPS73633:TPS73633DBVTG4
- added U9: TXB0104, SparkFun-IC-Comms:TXB0104PWR
- added X1: WIFI_1, adafruit:SMACONNECTOR_EDGE
- added X2: WIFI_2, adafruit:SMACONNECTOR_EDGE
Connections:
- new net +12V: PS1.+VOUT, R7.2, TP3.1, U$2.VOUT+, U5.IN+, U5.VBUS
- new net +3V3: C1.1, C11.1, C14.1, C15.1, C2.1, C4.1, C7.1, C9.1, R12.2, R13.2, R14.2, TP4.1, U$1.3V3, U1.CSB, U1.VDD, U1.VDDIO, U2.A0, U2.A1, U2.VDD, U3.VCCB, U4.VDD, U6.VCCB, U7.OUT, U8.VCCB
- new net CS: J8.3, U9.B2
- new net EXT_VIN: D9.C, F1.2, J5-1.S
- new net MISO: J8.4, U9.B3
- new net MOSI: J8.5, U9.B4
- new net N$1: D7.C, R5.1, U5.ALERT
- new net N$10: ANT2.SIG, X2.ANT
- new net N$11: D6.R_A, R21.1
- new net N$12: ANT2.GND1, ANT2.GND2, X2.GND1, X2.GND2, X2.GND3, X2.GND4
- new net N$13: D5.A, R7.1
- new net N$14: ANT1.GND1, ANT1.GND2, X1.GND1, X1.GND2, X1.GND3, X1.GND4
- new net N$15: D8.A, R8.1
- new net N$16: C19.1, U7.NR/FB
- new net N$17: D10.A, R12.1
- new net N$2: ANT1.SIG, X1.ANT
- new net N$21: D1.C, U2.LED0
- new net N$22: D2.C, U2.LED1
- new net N$23: J3.2, U3.B1
- new net N$24: J3.3, U3.B2
- new net N$25: D4.C, U2.LED2
- new net N$26: D3.C, U2.LED3
- new net N$27: F1.1, PS1.+VIN, TP2.1, U$2.EN, U$2.VIN
- new net N$28: D6.B_C, U4.LED2
- new net N$29: D6.G_C, U4.LED1
- new net N$3: D1.A, R15.1
- new net N$30: D6.R_C, U4.LED0
- new net N$31: J4.2, U8.B1
- new net N$34: J4.3, U8.B2
- new net N$4: D2.A, R16.1
- new net N$5: D4.A, R17.1
- new net N$6: D3.A, R18.1
- new net N$7: D7.A, R6.2
- new net N$8: D6.B_A, R19.1
- new net N$9: D6.G_A, R20.1
- new net SCLK: J8.2, U9.B1
- new net SCL_3V3: J6.2, J7.2, R13.1, TP7.1, U$1.SCL, U1.SCLK, U2.SCL, U4.SCL, U5.SCL, U6.B2
- new net SDA_3V3: J6.3, J7.3, R14.1, TP6.1, U$1.SDA, U1.SDI, U2.SDA, U4.SDA, U5.SDA, U6.B1
- net +1V8: now also C10.1, C12.1, C6.1, C8.1, R1.2, R10.2, R11.2, R2.2, R3.2, R4.2, R9.2, TP1.1, U3.OE, U3.VCCA, U6.OE, U6.VCCA, U8.OE, U8.VCCA, U9.OE, U9.VCCA
- net +5V: now also C13.1, C3.1, C5.1, J3.1, J4.1, J6.1, J7.1, J8.1, R15.2, R16.2, R17.2, R18.2, R19.2, R20.2, R21.2, R5.2, R6.1, TP5.1, U5.VS, U7.EN, U7.IN, U9.VCCB
- net GND: now also C1.2, C10.2, C11.2, C12.2, C13.2, C14.2, C15.2, C16.2, C17.2, C18.2, C19.2, C2.2, C3.2, C4.2, C5.2, C6.2, C7.2, C8.2, C9.2, D10.C, D5.C, D8.C, D9.A, J3.4, J3.SHIELD, J4.4, J4.SHIELD, J5-2.S, J6.4, J6.SHIELD, J7.4, J7.SHIELD, J8.6, J8.SHIELD, PS1.GND, S1.GND, S2.2, U$1.GND, U$2.VIN-, U$2.VOUT-, U1.GND, U1.SDO, U2.VSS, U4.A0, U4.A1, U4.VSS, U5.A0, U5.A1, U5.GND, U6.GND, U7.GND, U9.GND
- net GPIO-G: now also R10.1, S1.RIGHT
- net GPIO-I: now also R9.1, S1.LEFT
- net GPIO-J: now also R4.1, S1.DOWN
- net GPIO-K: now also R3.1, S1.UP
- net GPIO-L: now also R11.1, S1.CENT
- net I2C1_SCL: now also R1.1, U6.A2
- net I2C1_SDA: now also R2.1, U6.A1
- net RST_BTN_N: now also S2.1
- net SPI0_CS: now also U9.A2
- net SPI0_DIN: now also U9.A3
- net SPI0_DOUT: now also U9.A1
- net SPI0_SCLK: now also U9.A4
- net SYS_DCIN: now also C16.1, C17.1, C18.1, R8.2, U5.IN-
- net UART0_RXD: now also U3.A2
- net UART0_TXD: now also U3.A1
- net UART1_RXD: now also U8.A2
- net UART1_TXD: now also U8.A1
Other:
- note added: "0x3C"
- note added: "1.8V to 3.3V Conversion"
- note added: "5V Power, 3V logic"
- note added: "5V to 3V LDO"
- note added: "96Boards typically have pullups on GPIOs, resistors here for safety"
- note added: "ACTIVE LOW"
- note added: "AUTOPILOT"
- note added: "Address: 0b1000000"
- note added: "Address: 0b1100000"
- note added: "Address: 0b1100011"
- note added: "Address: 0b1110111"
- note added: "Display"
- note added: "Environmental Sensors"
- note added: "External In"
- note added: "External to 12V Conversion"
- note added: "I2C Devices"
- note added: "LED Controllers"
- note added: "No connect 5V power for PX4 Connection"
- note added: "Note: 5V power supply, 3V3 Logic"
- note added: "Optical Module"
- note added: "Particulate Sensor"
- note added: "Power Indication"
- note added: "Power Monitoring"
- note added: "Power Supplies"
- note added: "RADIO"
- note added: "Sensors/Outputs"
- note added: "The RFD-868 radios require 5V power, but 3V3 signalling."
- note added: "UART Connections for Autpilot and Radio"
- note added: "UART0 is by default set to console output - disable this."
- note added: "WiFi Antennas"
